File: mainboard/DCO.sch (EAGLE design)
At the start: 44 parts, among them IC101 LF353D, IC201 LF353D, IC301 V_REG_MIC2920, J3 M04X2, P101 TRIMPOT 100K, U1 XMEGA-A4VQFN

Commit message: rerouted, switched to TQFP xmega
Parts:
- added TP105: M01PTH, SparkFun:M01PTH
- R102: value 3.9 -> 1
- U1: value XMEGA-A4VQFN -> XMEGA-A4TQFP; device custom:XMEGA-A4VQFN -> avr-7:XMEGA-A4TQFP
Connections:
- net FREQCV: now also TP103.1
- net N$13: now also TP105.1; no longer TP104.1
- net N$5: now also TP104.1; no longer TP103.1
Other:
- moved on the sheet: TP103, TP104
Changed lines of the file:
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@@
 <?xml version="1.0" encoding="utf-8"?>
 <!DOCTYPE eagle SYSTEM "eagle.dtd">
-<eagle version="6.1">
+<eagle version="6.4">
 <drawing>
 <settings>
@@
 <setting verticaltext="up"/>
 </settings>
-<grid distance="0.1" unitdist="inch" unit="inch" style="lines" multiple="1" display="no" altdistance="0.01" altunitdist="inch" altunit="inch"/>
+<grid distance="0.05" unitdist="inch" unit="inch" style="lines" multiple="1" display="yes" altdistance="0.01" altunitdist="inch" altunit="inch"/>
 <layers>
 <layer number="1" name="Top" color="4" fill="1" visible="no" active="no"/>
@@
 <part name="Q101" library="SparkFun" deviceset="TRANSISTOR_NPN" device="SOT23"/>
 <part name="C101" library="SparkFun" deviceset="CAP" device="0603-CAP" value="220pF"/>
-<part name="R102" library="SparkFun" deviceset="RESISTOR" device="0805-RES" value="3.9"/>
+<part name="R102" library="SparkFun" deviceset="RESISTOR" device="0805-RES" value="1"/>
 <part name="GND2" library="supply1" deviceset="GND" device=""/>
 <part name="C103" library="SparkFun" deviceset="CAP" device="0805" value="1uF"/>
@@
 <part name="TP101" library="SparkFun" deviceset="M01" device="PTH" value=""/>
 <part name="TP102" library="SparkFun" deviceset="M01" device="PTH" value=""/>
+<part name="TP105" library="SparkFun" deviceset="M01" device="PTH" value=""/>
 <part name="TP104" library="SparkFun" deviceset="M01" device="PTH" value=""/>
-<part name="TP103" library="SparkFun" deviceset="M01" device="PTH" value=""/>
 <part name="R101" library="SparkFun" deviceset="RESISTOR" device="0603-RES" value="10K"/>
 <part name="GND5" library="supply1" deviceset="GND" device=""/>
@@
 <part name="P+6" library="supply1" deviceset="+5V" device=""/>
 <part name="GND12" library="SparkFun" deviceset="GND" device=""/>
-<part name="U1" library="custom" deviceset="XMEGA-A4" device="VQFN"/>
+<part name="U1" library="avr-7" deviceset="XMEGA-A4" device="TQFP"/>
 <part name="+3V2" library="supply1" deviceset="+3V3" device=""/>
 <part name="GND11" library="supply1" deviceset="GND" device=""/>
@@
 <part name="P-1" library="supply1" deviceset="-5V" device=""/>
 <part name="C304" library="SparkFun" deviceset="CAP" device="1206" value="10uF"/>
+<part name="TP103" library="SparkFun" deviceset="M01" device="PTH" value=""/>
 </parts>
 <sheets>
@@
 <instance part="TP101" gate="G$1" x="7.62" y="146.05"/>
 <instance part="TP102" gate="G$1" x="26.67" y="162.56"/>
-<instance part="TP104" gate="G$1" x="93.98" y="133.35" rot="R90"/>
-<instance part="TP103" gate="G$1" x="52.07" y="133.35" rot="R90"/>
+<instance part="TP105" gate="G$1" x="93.98" y="133.35" rot="R90"/>
+<instance part="TP104" gate="G$1" x="52.07" y="133.35" rot="R90"/>
 <instance part="R101" gate="G$1" x="15.24" y="137.16" rot="R90"/>
 <instance part="GND5" gate="1" x="15.24" y="127"/>
@@
 </instance>
 <instance part="C304" gate="G$1" x="35.56" y="29.21"/>
+<instance part="TP103" gate="G$1" x="50.8" y="170.18" rot="R180"/>
 </instances>
 <busses>
@@
 <segment>
 <pinref part="R103" gate="G$1" pin="2"/>
-<wire x1="39.37" y1="168.91" x2="39.37" y2="172.72" width="0.1524" layer="91"/>
+<wire x1="39.37" y1="168.91" x2="39.37" y2="170.18" width="0.1524" layer="91"/>
+<wire x1="39.37" y1="170.18" x2="39.37" y2="172.72" width="0.1524" layer="91"/>
 <wire x1="39.37" y1="172.72" x2="33.02" y2="172.72" width="0.1524" layer="91"/>
 <label x="33.02" y="172.72" size="1.778" layer="95"/>
+<pinref part="TP103" gate="G$1" pin="1"/>
+<wire x1="39.37" y1="170.18" x2="43.18" y2="170.18" width="0.1524" layer="91"/>
+<junction x="39.37" y="170.18"/>
 </segment>
 <segment>
@@
 <wire x1="52.07" y1="153.67" x2="52.07" y2="140.97" width="0.1524" layer="91"/>
 <junction x="52.07" y="153.67"/>
-<pinref part="TP103" gate="G$1" pin="1"/>
+<pinref part="TP104" gate="G$1" pin="1"/>
 </segment>
 </net>
@@
 <pinref part="R106" gate="G$1" pin="2"/>
 <wire x1="83.82" y1="147.32" x2="93.98" y2="147.32" width="0.1524" layer="91"/>
-<pinref part="TP104" gate="G$1" pin="1"/>
+<pinref part="TP105" gate="G$1" pin="1"/>
 <wire x1="93.98" y1="140.97" x2="93.98" y2="147.32" width="0.1524" layer="91"/>
 <wire x1="93.98" y1="156.21" x2="93.98" y2="147.32" width="0.1524" layer="91"/>

Commit message: Fixed design flaw - these resistors should be 10K
Parts:
- R301, R302: value 100K -> 10K
Changed lines of the file:
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@@
 <part name="D302" library="SparkFun" deviceset="DIODE-ZENER" device="-BZT52" value="5V"/>
 <part name="GND10" library="supply1" deviceset="GND" device=""/>
-<part name="R301" library="SparkFun" deviceset="RESISTOR" device="0603-RES" value="100K"/>
-<part name="R302" library="SparkFun" deviceset="RESISTOR" device="0603-RES" value="100K"/>
+<part name="R301" library="SparkFun" deviceset="RESISTOR" device="0603-RES" value="10K"/>
+<part name="R302" library="SparkFun" deviceset="RESISTOR" device="0603-RES" value="10K"/>
 <part name="P+5" library="supply1" deviceset="+12V" device=""/>
 <part name="P-4" library="supply1" deviceset="-12V" device=""/>
